Commit message: working on gazebo

File: description/robot_core.xacro (robot description, xacro)
@@ -143,26 +143,118 @@
     </link>
         <!-- Chassis Aufbau-->
-        <joint name="chassis_joint" type="fixed">
-            <parent link="base_link"/>
-            <child link="body"/>
-            <origin xyz="-0.08 0.0 0.055"/>
-        </joint>
-        <link name="body">
-            <visual>
-                <origin xyz="0.0 0.0 0.0" rpy="0.0 0.0 0.0"/>
-                <geometry>
-                    <box size="0.4 0.11 0.07"/>
-                </geometry>
-                <material name="orange"/>
-            </visual>
-            <collision>
-                <origin xyz="0.0 0.0 0.003" rpy="0.0 0.0 0.0"/>
-                <geometry>
-                    <box size="0.4 0.11 0.07"/>
-                </geometry>
-            </collision>
-            <xacro:inertial_box mass="0.2" x="0.4" y="0.11" z="0.07">
-                <origin xyz="0.0 0.0 0.003" rpy="0.0 0.0 0.0"/>
-            </xacro:inertial_box>
-         </link>
+    <joint name="chassis_joint" type="fixed">
+        <parent link="base_link"/>
+        <child link="body"/>
+        <origin xyz="-0.08 0.0 0.055"/>
+    </joint>
+    <link name="body">
+        <visual>
+            <origin xyz="0.0 0.0 0.0" rpy="0.0 0.0 0.0"/>
+            <geometry>
+                <box size="0.4 0.11 0.07"/>
+            </geometry>
+            <material name="orange"/>
+        </visual>
+        <collision>
+            <origin xyz="0.0 0.0 0.003" rpy="0.0 0.0 0.0"/>
+            <geometry>
+                <box size="0.4 0.11 0.07"/>
+            </geometry>
+        </collision>
+        <xacro:inertial_box mass="0.2" x="0.4" y="0.11" z="0.07">
+            <origin xyz="0.0 0.0 0.003" rpy="0.0 0.0 0.0"/>
+        </xacro:inertial_box>
+     </link>
+     <joint name="body_joint" type="fixed">
+        <parent link="body"/>
+        <child link="body_top"/>
+        <origin xyz="0 0.0 0.07"/>
+    </joint>
+    <link name="body_top">
+        <visual>
+            <origin xyz="-0.04 0.0 0.0" rpy="0.0 0.0 0.0"/>
+            <geometry>
+                <box size="0.32 0.11 0.07"/>
+            </geometry>
+            <material name="orange"/>
+        </visual>
+        <collision>
+            <origin xyz="0.0 0.0 0.0" rpy="0.0 0.0 0.0"/>
+            <geometry>
+                <box size="0.4 0.11 0.07"/>
+            </geometry>
+        </collision>
+        <xacro:inertial_box mass="0.2" x="0.4" y="0.11" z="0.07">
+            <origin xyz="0.0 0.0 0.0" rpy="0.0 0.0 0.0"/>
+        </xacro:inertial_box>
+     </link>
+     <!-- Cam-->
+     <joint name="cam_joint" type="fixed">
+        <parent link="body"/>
+        <child link="cam"/>
+        <origin xyz="0.17 0 0.07 "/>
+    </joint>
+    <link name="cam">
+        <visual>
+            <origin xyz="0.0 0.0 0.0" rpy="0.0 0.0 0.0"/>
+            <geometry>
+                <box size="0.04 0.11 0.07"/>
+            </geometry>
+            <material name="white"/>
+        </visual>
+        <collision>
+            <origin xyz="0.0 0.0 0.0" rpy="0.0 0.0 0.0"/>
+            <geometry>
+                <box size="0.4 0.11 0.07"/>
+            </geometry>
+        </collision>
+        <xacro:inertial_box mass="0.2" x="0.04" y="0.11" z="0.07">
+            <origin xyz="0.0 0.0 0.0" rpy="0.0 0.0 0.0"/>
+        </xacro:inertial_box>
+     </link>
+     <!-- LIDAR-->
+     <joint name="li_top_joint" type="fixed">
+        <parent link="body_top"/>
+        <child link="li_top"/>
+        <origin xyz="0.075 0 0.047 "/>
+    </joint>
+    <link name="li_top">
+        <visual>
+            <origin xyz="0.0 0.0 0.0" rpy="0.0 0.0 0.0"/>
+            <geometry>
+                <box size="0.04 0.11 0.025"/>
+            </geometry>
+            <material name="black"/>
+        </visual>
+        <collision>
+            <origin xyz="0.0 0.0 0.0" rpy="0.0 0.0 0.0"/>
+            <geometry>
+                <box size="0.4 0.11 0.025"/>
+            </geometry>
+        </collision>
+        <xacro:inertial_box mass="0.2" x="0.04" y="0.11" z="0.025">
+            <origin xyz="0.0 0.0 0.0" rpy="0.0 0.0 0.0"/>
+        </xacro:inertial_box>
+     </link>
+     <joint name="lidar_joint" type="fixed">
+        <origin xyz="0.0 0.0 0.03" rpy="-0.0 0.0 0.0"/>
+        <parent link="li_top"/>
+        <child link="lidar"/>
+    </joint>
+    <link name="lidar">
+        <visual>
+            <geometry>
+                <cylinder radius="0.06" length="0.04"/>
+            </geometry>
+            <material name="blue"/>
+        </visual>
+        <collision>
+            <geometry>
+                <sphere radius="0.06"/>
+            </geometry>
+        </collision>
+        <xacro:inertial_cylinder mass="0.01" radius="0.06" length="0.04">
+            <origin xyz="0.0 0.0 0.0" rpy="0.0 0.0 0.0"/>
+        </xacro:inertial_cylinder>
+    </link>
 </robot>

Commit message: play with scout

File: description/robot_core.xacro (robot description, xacro)
@@ -24,4 +24,13 @@
         <color rgba="1.0 0.0 0.0 1.0"/>
     </material>
+    <!-- BASE_FOOT_PRINT-->
+    <link name="base_footprint">
+    </link>
+    <!-- FOOTPRINT JOINT -->
+    <joint name="basefootprint_joint" type="fixed">
+        <parent link="base_link"/>
+        <child link="base_footprint"/>
+        <origin xyz="0.0 0.0 0.0"/>
+    </joint>
     <!-- BASE LINK -->
     <link name="base_link">
