Commit message: lidar works

File: description/lidar.xacro (robot description, xacro)
@@ -31,7 +31,7 @@
        <origin xyz="0.0 0.0 0.03" rpy="0.0 0.0 1.57"/>
        <parent link="li_top"/>
-       <child link="lidar"/>
+       <child link="laser_frame"/>
     </joint>
-    <link name="lidar">
+    <link name="laser_frame">
         <visual>
             <geometry>
@@ -49,6 +49,9 @@
         </xacro:inertial_cylinder>
     </link>
+    <gazebo reference="laser_frame">
+        <material>Gazebo/Red</material>
+    </gazebo>
         <!-- Gazebo Plugin-->
-    <gazebo reference="lidar">
+    <gazebo reference="laser_frame">
         <material>Gazebo/Red</material>
         <sensor name="laser" type="ray">
@@ -68,10 +71,9 @@
                     <min>0.3</min>
                     <max>12</max>
-                    <resolution>0.01</resolution>
                 </range>
             </ray>
             <plugin name="laser_controller" filename="libgazebo_ros_ray_sensor.so">
                 <ros>
-                    <argument>~/out:=scan</argument> <!-- - -ros-args - -remap ~ -->
+                    <argument>~/out:=scan</argument>
                 </ros>
                 <output_type>sensor_msgs/LaserScan</output_type>

Commit message: restart urdf

File: description/lidar.xacro (robot description, xacro)
@@ -57,5 +57,5 @@
         <sensor name="laser" type="ray">
             <pose> 0 0 0 0 0 0 </pose>
-            <visualize>false</visualize>
+            <visualize>true</visualize>
             <update_rate>10</update_rate>
             <ray>

File: description/robot.urdf.xacro (robot description, xacro)
@@ -1,7 +1,8 @@
 <?xml version="1.0"?>
-<robot xmlns:xacro="http://www.ros.org/wiki/xacro"  name="homebot">
+<robot xmlns:xacro="http://www.ros.org/wiki/xacro"  name="scout">
+    <xacro:include filename="scout_core.xacro"/>
+<!--
     <xacro:arg name="use_ros2_control" default="false"/>
     <xacro:arg name="sim_mode" default="true"/>
-    <xacro:include filename="robot_core.xacro"/>
     <xacro:if value="$(arg use_ros2_control)">
         <xacro:include filename="ros2_control.xacro"/>
@@ -12,3 +13,4 @@
     <xacro:include filename="lidar.xacro"/>
     <xacro:include filename="camera.xacro"/>
+-->
 </robot>

File: description/robot_core.xacro (robot description, xacro)
@@ -92,8 +92,8 @@
     <!-- RIGHT WHEEL  LINK -->
     <joint name="right_wheel_joint" type="continuous">
-        <origin xyz="0 0.128 0.017" rpy="-${pi/2} 0 0"/>
+        <origin xyz="0 0.128 0.017" rpy="${pi/2} 0 0"/>
         <parent link="base_link"/>
         <child link="right_wheel"/>
-        <axis xyz="0.0 0.0 -1.0"/>
+        <axis xyz="0.0 0.0 1.0"/>
         <limit lower="0.0" upper="0.0" effort="0.0" velocity="0.0"/>
     </joint>
