Commit message: urdf base works

File: description/scout_core.xacro (robot description, xacro)
@@ -31,9 +31,9 @@
         <parent link="base_link"/>
         <child link="chassis"/>
-        <origin xyz="-0.017 0.0 0.0"/>
+        <origin xyz="-0.26 0.0 0.0"/>
     </joint>
     <link name="chassis">
         <visual>
-            <origin xyz="0.017 0.0 0.017"/>
+            <origin xyz="0.26 0.0 0.017"/>
             <geometry>
                 <box size="0.034 0.25 0.034"/>
@@ -42,10 +42,10 @@
         </visual>
         <collision>
-            <origin xyz="0.093 0.0 0.075"/>
+            <origin xyz="0.26 0.0 0.017"/>
             <geometry>
                 <box size="0.034 0.25 0.034"/>
             </geometry>
         </collision>
-        <xacro:inertial_box mass="1.5" x="0.034" y="0.25" z="0.034">
+        <xacro:inertial_box mass="0.5" x="0.034" y="0.25" z="0.034">
             <origin xyz="0.0 0.0 0.0" rpy="0.0 0.0 0.0"/>
         </xacro:inertial_box>
@@ -54,3 +54,112 @@
         <material>Gazebo/Black</material>
     </gazebo>
+    <!-- LEFT WHEEL LINK -->
+    <joint name="left_wheel_joint" type="continuous">
+        <origin xyz="0 -0.148 0.017" rpy="-${pi/2} 0 0"/>
+        <parent link="base_link"/>
+        <child link="left_wheel"/>
+        <axis xyz="0.0 0.0 1.0"/>
+        <limit lower="0.0" upper="0.0" effort="0.0" velocity="0.0"/>
+    </joint>
+    <link name="left_wheel">
+        <visual>
+            <geometry>
+                <cylinder radius="0.06" length="0.04"/>
+            </geometry>
+            <material name="blue"/>
+        </visual>
+        <collision>
+            <geometry>
+                <sphere radius="0.06"/>
+            </geometry>
+        </collision>
+        <xacro:inertial_sphere mass="0.3" radius="0.06">
+            <origin xyz="0.0 0.0 0.0" rpy="0.0 0.0 0.0"/>
+        </xacro:inertial_sphere>
+    </link>
+    <gazebo reference="left_wheel">
+        <material>Gazebo/Blue</material>
+    </gazebo>
+    <!-- RIGHT WHEEL LINK -->
+    <joint name="right_wheel_joint" type="continuous">
+        <origin xyz="0 0.148 0.017" rpy="${pi/2} 0 0"/>
+        <parent link="base_link"/>
+        <child link="right_wheel"/>
+        <axis xyz="0.0 0.0 -1.0"/>
+        <limit lower="0.0" upper="0.0" effort="0.0" velocity="0.0"/>
+    </joint>
+    <link name="right_wheel">
+        <visual>
+            <geometry>
+                <cylinder radius="0.06" length="0.04"/>
+            </geometry>
+            <material name="blue"/>
+        </visual>
+        <collision>
+            <geometry>
+                <sphere radius="0.06"/>
+            </geometry>
+        </collision>
+        <xacro:inertial_sphere mass="0.3" radius="0.06">
+            <origin xyz="0.0 0.0 0.0" rpy="0.0 0.0 0.0"/>
+        </xacro:inertial_sphere>
+    </link>
+    <gazebo reference="right_wheel">
+        <material>Gazebo/Blue</material>
+    </gazebo>
+    <!-- Caster Wheel Holder and Caster Wheel -->
+    <joint name="caster_wheel_holder_joint" type="fixed">
+        <parent link="base_link"/>
+        <child link="caster_wheel_holder"/>
+        <origin xyz="-0.22 0.0 0.0"/>
+    </joint>
+    <link name="caster_wheel_holder">
+        <visual>
+            <origin xyz="0.0 0.0 0.017"/>
+            <geometry>
+                <box size="0.034 0.034 0.034"/>
+            </geometry>
+            <material name="black"/>
+        </visual>
+        <collision>
+            <origin xyz="0.0 0.0 0.017"/>
+            <geometry>
+                <box size="0.034 0.034 0.034"/>
+            </geometry>
+        </collision>
+        <xacro:inertial_box mass="1.5" x="0.034" y="0.034" z="0.034">
+            <origin xyz="0.0 0.0 0.0" rpy="0.0 0.0 0.0"/>
+        </xacro:inertial_box>
+    </link>
+    <gazebo reference="caster_wheel_holder">
+        <material>Gazebo/Black</material>
+    </gazebo>
+    <!-- caster Wheel-->
+    <joint name="caster_wheel_joint" type="fixed">
+        <parent link="caster_wheel_holder"/>
+        <child link="caster_wheel_link"/>
+        <origin xyz="0.0 0.0 -0.017"/>
+    </joint>
+    <link name="caster_wheel_link">
+        <visual>
+            <geometry>
+                <sphere radius="0.03"/>
+            </geometry>
+            <material name="blue">
+            </material>
+        </visual>
+        <collision>
+            <geometry>
+                <sphere radius="0.03"/>
+            </geometry>
+        </collision>
+        <xacro:inertial_sphere mass="0.15" radius="0.03">
+            <origin xyz="0.0 0.0 0.0" rpy="0.0 0.0 0.0"/>
+        </xacro:inertial_sphere>
+    </link>
+    <gazebo reference="caster_wheel_link">
+        <material>Gazebo/Blue</material>
+        <mu1 value="0.001"/>
+        <mu2 value="0.001"/>
+    </gazebo>
 </robot>
