Commit message: save this

File: description/gazebo_control.xacro (robot description, xacro)
@@ -3,13 +3,13 @@
     <gazebo>
         <plugin name="diff_drive" filename="libgazebo_ros_diff_drive.so">
-            <!-- Wheel Information -->
+            <!-- Reifen Infos -->
             <left_joint>left_wheel_joint</left_joint>
             <right_joint>right_wheel_joint</right_joint>
-            <wheel_separation>0.25</wheel_separation>
-            <wheel_diameter>0.06</wheel_diameter>
-            <!-- Limits -->
+            <wheel_separation>0.35</wheel_separation>
+            <wheel_diameter>0.12</wheel_diameter>
+            <!-- LIMITS       -->
             <max_wheel_torque>200</max_wheel_torque>
             <max_wheel_acceleration>10.0</max_wheel_acceleration>
-            <!-- Output -->
+            <!-- Output       -->
             <odometry_frame>odom</odometry_frame>
             <robot_base_frame>base_link</robot_base_frame>

File: description/lidar.xacro (robot description, xacro)
@@ -5,5 +5,5 @@
         <parent link="body_top"/>
         <child link="li_top"/>
-        <origin xyz="0.075 0 0.047 "/>
+        <origin xyz="-0.12 0 0.047 "/>
     </joint>
     <link name="li_top">
@@ -49,6 +49,33 @@
         </xacro:inertial_cylinder>
     </link>
+        <!-- Gazebo Plugin-->
     <gazebo reference="lidar">
         <material>Gazebo/Red</material>
+        <sensor name="laser" type="ray">
+            <pose> 0 0 0 0 0 0 </pose>
+            <visualize>true</visualize>
+            <update_rate>10</update_rate>
+            <ray>
+                <scan>
+                    <horizontal>
+                        <samples>360</samples>
+                        <resolution>1</resolution>
+                        <min_angle>0.00</min_angle>
+                        <max_angle>3.14</max_angle>
+                    </horizontal>
+                </scan>
+                <range>
+                    <min>0.3</min>
+                    <max>8</max>
+                </range>
+            </ray>
+            <plugin name="laser_controller" filename="libgazebo_ros_ray_sensor.so">
+                <ros>
+                    <argument>~/out:=scan</argument>
+                </ros>
+                <output_type>sensor_msgs/LaserScan</output_type>
+                <frame_name>laser_frame</frame_name>
+            </plugin>
+        </sensor>
     </gazebo>
 </robot>

File: description/robot.urdf.xacro (robot description, xacro)
@@ -1,9 +1,14 @@
 <?xml version="1.0"?>
-<robot xmlns:xacro="http://www.ros.org/wiki/xacro"  name="scout">
+<robot xmlns:xacro="http://www.ros.org/wiki/xacro"  name="homebot">
+    <xacro:arg name="use_ros2_control" default="false"/>
+    <xacro:arg name="sim_mode" default="true"/>
     <xacro:include filename="robot_core.xacro"/>
-    <!--
+    <xacro:if value="$(arg use_ros2_control)">
+        <xacro:include filename="ros2_control.xacro"/>
+    </xacro:if>
+    <xacro:unless value="$(arg use_ros2_control)">
+        <xacro:include filename="gazebo_control.xacro"/>
+    </xacro:unless>
+    <xacro:include filename="lidar.xacro"/>
     <xacro:include filename="camera.xacro"/>
-    <xacro:include filename="lidar.xacro"/>
-    -->
-    <xacro:include filename="gazebo_control.xacro"/>
 </robot>

File: description/robot_core.xacro (robot description, xacro)
@@ -1,6 +1,6 @@
 <?xml version="1.0"?>
-<robot xmlns:xacro="http://www.ros.org/wiki/xacro" >
+<robot xmlns:xacro="http://www.ros.org/wiki/xacro">
     <xacro:include filename="inertial_macros.xacro"/>
-    <!-- FARBEN in RotGrünBlauAmber-->
+            <!-- Farben -->
     <material name="white">
         <color rgba="1 1 1 1"/>
@@ -21,28 +21,26 @@
         <color rgba="0.0 1.0 0.0 1.0"/>
     </material>
-    <material name="LightGrey">
-        <color rgba="0.7 0.7 0.7 1.0"/>
-    </material>
     <material name="red">
-        <color rgba="1 0. 0. 1.0"/>
+        <color rgba="1.0 0.0 0.0 1.0"/>
     </material>
     <!-- BASE LINK -->
-    <link name="base_link"/>
-    <!-- Chassis Link AKA Rad Strebe-->
-    <joint name="chassis_joint" type="fixed">
+    <link name="base_link">
+    </link>
+    <!-- CHASSIS LINK -->
+    <joint name="cassis_joint" type="fixed">
         <parent link="base_link"/>
         <child link="chassis"/>
-        <origin xyz="0.0 0.0 0.0"/>
+        <origin xyz="-0.017 0.0 0.0"/>
     </joint>
     <link name="chassis">
         <visual>
-            <origin xyz="0.0 0.0 0.003" rpy="0.0 0.0 0.0"/>
+            <origin xyz="0.017 0.0 0.017"/>
             <geometry>
                 <box size="0.034 0.25 0.034"/>
             </geometry>
-            <material name="black"/>
-        </visual>
-        <collision>
-            <origin xyz="0.0 0.0 0.003" rpy="0.0 0.0 0.0"/>
+            <material name="orange"/>
+        </visual>
+        <collision>
+            <origin xyz="0.093 0.0 0.075"/>
             <geometry>
                 <box size="0.034 0.25 0.034"/>
@@ -56,94 +54,98 @@
         <material>Gazebo/Black</material>
     </gazebo>
-    <joint name="chassi_t_joint" type="fixed">
-       <parent link="chassis"/>
-       <child link="chassis_t"/>
-       <origin xyz="-0.12 0.0 0.0"/>
-    </joint>
-    <link name="chassis_t">
-        <visual>
-            <origin xyz="0.0 0.0 0.003" rpy="0.0 0.0 -${pi/2}"/>
-            <geometry>
-                <box size="0.034 0.25 0.034"/>
+        <!-- LEFT WHEEL LINK -->
+    <joint name="left_wheel_joint" type="continuous">
+        <origin xyz="0 -0.128 0.017" rpy="${pi/2} 0 0"/>
+        <parent link="base_link"/>
+        <child link="left_wheel"/>
+        <axis xyz="0.0 0.0 1.0"/>
+        <limit lower="0.0" upper="0.0" effort="0.0" velocity="0.0"/>
+    </joint>
+    <link name="left_wheel">
+        <visual>
+            <geometry>
+                <cylinder radius="0.06" length="0.04"/>
+            </geometry>
+            <material name="blue"/>
+        </visual>
+        <collision>
+            <geometry>
+                <cylinder radius="0.06" length="0.04"/>
+            </geometry>
+        </collision>
+        <xacro:inertial_cylinder mass="0.1" length="0.04" radius="0.06">
+            <origin xyz="0.0 0.0 0.0" rpy="0.0 0.0 0.0"/>
+        </xacro:inertial_cylinder>
+    </link>
+    <gazebo reference="left_wheel">
+        <material>Gazebo/Blue</material>
+    </gazebo>
+    <!-- RIGHT WHEEL  LINK -->
+    <joint name="right_wheel_joint" type="continuous">
+        <origin xyz="0 0.128 0.017" rpy="-${pi/2} 0 0"/>
+        <parent link="base_link"/>
+        <child link="right_wheel"/>
+        <axis xyz="0.0 0.0 -1.0"/>
+        <limit lower="0.0" upper="0.0" effort="0.0" velocity="0.0"/>
+    </joint>
+    <link name="right_wheel">
+        <visual>
+            <geometry>
+                <cylinder radius="0.06" length="0.04"/>
+            </geometry>
+            <material name="blue"/>
+        </visual>
+        <collision>
+            <geometry>
+                <cylinder radius="0.06" length="0.04"/>
+            </geometry>
+        </collision>
+        <xacro:inertial_cylinder mass="0.1" length="0.04" radius="0.06">
+            <origin xyz="0.0 0.0 0.0" rpy="0.0 0.0 0.0"/>
+        </xacro:inertial_cylinder>
+    </link>
+    <gazebo reference="right_wheel">
+        <material>Gazebo/Blue</material>
+    </gazebo>
+    <!-- Caster Wheel Holder and Caster Wheel -->
+    <joint name="caster_wheel_holder_joint" type="fixed">
+        <parent link="chassis"/>
+        <child link="caster_wheel_holder"/>
+        <origin xyz="0.25 0.0 0.0"/>
+    </joint>
+    <link name="caster_wheel_holder">
+        <visual>
+            <origin xyz="0.0 0.0 0.017"/>
+            <geometry>
+                <box size="0.034 0.034 0.034"/>
             </geometry>
             <material name="black"/>
         </visual>
         <collision>
-            <origin xyz="0.0 0.0 0.003" rpy="0.0 0.0 0.0"/>
-            <geometry>
-                <box size="0.034 0.25 0.034"/>
-            </geometry>
-        </collision>
-        <xacro:inertial_box mass="1.5" x="0.034" y="0.25" z="0.034">
-            <origin xyz="0.0 0.0 0.0" rpy="0.0 0.0 0.0"/>
-        </xacro:inertial_box>
-    </link>
-    <gazebo reference="chassis_t">
+            <origin xyz="0.0 0.0 0.017"/>
+            <geometry>
+                <box size="0.034 0.034 0.034"/>
+            </geometry>
+        </collision>
+        <xacro:inertial_box mass="1.5" x="0.034" y="0.034" z="0.034">
+            <origin xyz="0.0 0.0 0.0" rpy="0.0 0.0 0.0"/>
+        </xacro:inertial_box>
+    </link>
+    <gazebo reference="caster_wheel_holder">
         <material>Gazebo/Black</material>
     </gazebo>
-    <!-- Linker Reifen-->
-    <joint name="left_wheel_joint" type="continuous">
-        <origin xyz="0.0 0.125 0.0" rpy="-${pi/2} 0.0 0.0"/>
-        <parent link="base_link"/>
-        <child link="left_wheel_link"/>
-        <axis xyz="0.0 0.0 1.0"/>
-    </joint>
-    <link name="left_wheel_link">
-        <visual>
-            <geometry>
-                <cylinder radius="0.06" length="0.04"/>
-            </geometry>
-            <material name="blue"/>
-        </visual>
-        <collision>
-            <geometry>
-                <cylinder radius="0.06" length="0.04"/>
-            </geometry>
-        </collision>
-        <xacro:inertial_cylinder mass="0.3" length="0.06" radius="0.04">
-            <origin xyz="0.0 0.0 0.0" rpy="0.0 0.0 0.0"/>
-        </xacro:inertial_cylinder>
-    </link>
-    <gazebo reference="left_wheel_link">
-        <material>Gazebo/Blue</material>
-    </gazebo>
-    <!-- Rechter Reifen-->
-    <joint name="right_wheel_joint" type="continuous">
-        <origin xyz="0.0 -0.125 0.0" rpy="-${pi/2} 0.0 0.0"/>
-        <parent link="base_link"/>
-        <child link="right_wheel_link"/>
-        <axis xyz="0.0 0.0 1.0"/>
-    </joint>
-    <link name="right_wheel_link">
-        <visual>
-            <geometry>
-                <cylinder radius="0.06" length="0.04"/>
-            </geometry>
-            <material name="blue"/>
-        </visual>
-        <collision>
-            <geometry>
-                <cylinder radius="0.06" length="0.04"/>
-            </geometry>
-        </collision>
-        <xacro:inertial_cylinder mass="0.3" length="0.06" radius="0.04">
-            <origin xyz="0.0 0.0 0.0" rpy="0.0 0.0 0.0"/>
-        </xacro:inertial_cylinder>
-    </link>
-    <gazebo reference="right_wheel_link">
-        <material>Gazebo/Blue</material>
-    </gazebo>
-    <!-- Caster Wheel Joint-->
+    <!-- caster Wheel-->
     <joint name="caster_wheel_joint" type="fixed">
-        <origin xyz="-0.23 0.0 -0.03" rpy="0.0 0.0 0.0"/>
-        <parent link="chassis"/>
-        <child link="caster_wheel"/>
-    </joint>
-    <link name="caster_wheel">
+        <parent link="caster_wheel_holder"/>
+        <child link="caster_wheel_link"/>
+        <origin xyz="0.0 0.0 -0.017"/>
+    </joint>
+    <link name="caster_wheel_link">
         <visual>
             <geometry>
                 <sphere radius="0.03"/>
             </geometry>
-            <material name="blue"/>
+            <material name="blue">
+            </material>
         </visual>
         <collision>
@@ -156,18 +158,18 @@
         </xacro:inertial_sphere>
     </link>
-    <gazebo reference="caster_wheel">
+    <gazebo reference="caster_wheel_link">
         <material>Gazebo/Blue</material>
         <mu1 value="0.001"/>
         <mu2 value="0.001"/>
     </gazebo>
-        <!-- Chassis Aufbau-->
-    <joint name="body_base_joint" type="fixed">
+    <!-- BODY PARTS-->
+    <joint name="body_joint" type="fixed">
         <parent link="chassis"/>
         <child link="body"/>
-        <origin xyz="-0.08 0.0 0.055"/>
+        <origin xyz="0.110 0.0 0.069"/>
     </joint>
     <link name="body">
         <visual>
-            <origin xyz="0.0 0.0 0.003" rpy="0.0 0.0 0.0"/>
+            <origin xyz="0.0 0.0 0.0"/>
             <geometry>
                 <box size="0.4 0.11 0.07"/>
@@ -176,10 +178,10 @@
         </visual>
         <collision>
-            <origin xyz="0.0 0.0 0.003" rpy="0.0 0.0 0.0"/>
+            <origin xyz="0.093 0.0 0.075"/>
             <geometry>
                 <box size="0.4 0.11 0.07"/>
             </geometry>
         </collision>
-        <xacro:inertial_box mass="0.2" x="0.4" y="0.11" z="0.07">
+        <xacro:inertial_box mass="0.5" x="0.4" y="0.11" z="0.07">
             <origin xyz="0.0 0.0 0.0" rpy="0.0 0.0 0.0"/>
         </xacro:inertial_box>
@@ -188,24 +190,25 @@
         <material>Gazebo/Orange</material>
     </gazebo>
-    <joint name="body_joint" type="fixed">
-        <parent link="body"/>
+    <!-- BodyTop-->
+    <joint name="body_top_joint" type="fixed">
+        <parent link="chassis"/>
         <child link="body_top"/>
-        <origin xyz="0 0.0 0.07"/>
+        <origin xyz="0.16 0.0 0.138"/>
     </joint>
     <link name="body_top">
         <visual>
-            <origin xyz="-0.04 0.0 0.0" rpy="0.0 0.0 0.0"/>
-            <geometry>
-                <box size="0.32 0.11 0.07"/>
+            <origin xyz="0.0 0.0 0.0"/>
+            <geometry>
+                <box size="0.3 0.11 0.07"/>
             </geometry>
             <material name="orange"/>
         </visual>
         <collision>
-            <origin xyz="-0.04 0.0 0.0" rpy="0.0 0.0 0.0"/>
-            <geometry>
-                <box size="0.32 0.11 0.07"/>
-            </geometry>
-        </collision>
-        <xacro:inertial_box mass="0.2" x="0.32" y="0.11" z="0.07">
+            <origin xyz="0.093 0.0 0.075"/>
+            <geometry>
+                <box size="0.4 0.11 0.07"/>
+            </geometry>
+        </collision>
+        <xacro:inertial_box mass="0.5" x="0.4" y="0.11" z="0.07">
             <origin xyz="0.0 0.0 0.0" rpy="0.0 0.0 0.0"/>
         </xacro:inertial_box>

Commit message: added Gazebo

File: description/gazebo_control.xacro (robot description, xacro)
@@ -6,5 +6,5 @@
             <left_joint>left_wheel_joint</left_joint>
             <right_joint>right_wheel_joint</right_joint>
-            <wheel_separation>0.36</wheel_separation>
+            <wheel_separation>0.3</wheel_separation>
             <wheel_diameter>0.12</wheel_diameter>
             <!-- LIMITS       -->

File: description/robot.urdf.xacro (robot description, xacro)
@@ -2,4 +2,5 @@
 <robot xmlns:xacro="http://www.ros.org/wiki/xacro"  name="scout">
     <xacro:include filename="scout_core.xacro"/>
+    <xacro:include filename="gazebo_control.xacro"/>
 <!--
     <xacro:arg name="use_ros2_control" default="false"/>

File: description/scout_core.xacro (robot description, xacro)
@@ -39,5 +39,5 @@
                 <box size="0.034 0.25 0.034"/>
             </geometry>
-            <material name="orange"/>
+            <material name="black"/>
         </visual>
         <collision>
@@ -47,5 +47,5 @@
             </geometry>
         </collision>
-        <xacro:inertial_box mass="0.5" x="0.034" y="0.25" z="0.034">
+        <xacro:inertial_box mass="1.5" x="0.034" y="0.25" z="0.034">
             <origin xyz="0.0 0.0 0.0" rpy="0.0 0.0 0.0"/>
         </xacro:inertial_box>
