Commit message: workflow

File: description/robot.urdf.xacro (robot description, xacro)
@@ -2,3 +2,5 @@
 <robot xmlns:xacro="http://www.ros.org/wiki/xacro"  name="scout">
     <xacro:include filename="robot_core.xacro"/>
+    <xacro:include filename="camera.xacro"/>
+    <xacro:include filename="lidar.xacro"/>
 </robot>

File: description/robot_core.xacro (robot description, xacro)
@@ -24,4 +24,7 @@
         <color rgba="0.7 0.7 0.7 1.0"/>
     </material>
+    <material name="red">
+        <color rgba="1 0. 0. 1.0"/>
+    </material>
     <!-- BASE LINK -->
     <link name="base_link">
@@ -29,7 +32,7 @@
     <!-- Chassis Link AKA Rad Strebe-->
     <joint name="chassis_joint" type="fixed">
-        <parent link="base_link"/>
-        <child link="chassis"/>
-        <origin xyz="0.1 0.0 0.0"/>
+        <parent link="chassis"/>
+        <child link="base_link"/>
+        <origin xyz="-0.0 0.0 0.0"/>
     </joint>
     <link name="chassis">
@@ -77,5 +80,5 @@
     <joint name="left_wheel_joint" type="continuous">
         <origin xyz="0.0 0.125 0.0" rpy="-${pi/2} 0.0 0.0"/>
-        <parent link="chassis"/>
+        <parent link="base_link"/>
         <child link="left_wheel"/>
         <axis xyz="0.0 0.0 1"/>
@@ -100,5 +103,5 @@
     <joint name="right_wheel_joint" type="continuous">
         <origin xyz="0.0 -0.125 0.0" rpy="-${pi/2} 0.0 0.0"/>
-        <parent link="chassis"/>
+        <parent link="base_link"/>
         <child link="right_wheel"/>
         <axis xyz="0.0 0.0 1"/>
@@ -123,5 +126,5 @@
     <joint name="caster_wheel_joint" type="fixed">
         <origin xyz="-0.23 0.0 -0.03" rpy="0.0 0.0 0.0"/>
-        <parent link="chassis"/>
+        <parent link="base_link"/>
         <child link="caster_wheel"/>
     </joint>
@@ -143,5 +146,5 @@
     </link>
         <!-- Chassis Aufbau-->
-    <joint name="chassis_joint" type="fixed">
+    <joint name="body_base_joint" type="fixed">
         <parent link="base_link"/>
         <child link="body"/>
@@ -189,72 +192,3 @@
         </xacro:inertial_box>
      </link>
-     <!-- Cam-->
-     <joint name="cam_joint" type="fixed">
-        <parent link="body"/>
-        <child link="cam"/>
-        <origin xyz="0.17 0 0.07 "/>
-    </joint>
-    <link name="cam">
-        <visual>
-            <origin xyz="0.0 0.0 0.0" rpy="0.0 0.0 0.0"/>
-            <geometry>
-                <box size="0.04 0.11 0.07"/>
-            </geometry>
-            <material name="white"/>
-        </visual>
-        <collision>
-            <origin xyz="0.0 0.0 0.0" rpy="0.0 0.0 0.0"/>
-            <geometry>
-                <box size="0.4 0.11 0.07"/>
-            </geometry>
-        </collision>
-        <xacro:inertial_box mass="0.2" x="0.04" y="0.11" z="0.07">
-            <origin xyz="0.0 0.0 0.0" rpy="0.0 0.0 0.0"/>
-        </xacro:inertial_box>
-     </link>
-     <!-- LIDAR-->
-     <joint name="li_top_joint" type="fixed">
-        <parent link="body_top"/>
-        <child link="li_top"/>
-        <origin xyz="0.075 0 0.047 "/>
-    </joint>
-    <link name="li_top">
-        <visual>
-            <origin xyz="0.0 0.0 0.0" rpy="0.0 0.0 0.0"/>
-            <geometry>
-                <box size="0.04 0.11 0.025"/>
-            </geometry>
-            <material name="black"/>
-        </visual>
-        <collision>
-            <origin xyz="0.0 0.0 0.0" rpy="0.0 0.0 0.0"/>
-            <geometry>
-                <box size="0.4 0.11 0.025"/>
-            </geometry>
-        </collision>
-        <xacro:inertial_box mass="0.2" x="0.04" y="0.11" z="0.025">
-            <origin xyz="0.0 0.0 0.0" rpy="0.0 0.0 0.0"/>
-        </xacro:inertial_box>
-     </link>
-     <joint name="lidar_joint" type="fixed">
-        <origin xyz="0.0 0.0 0.03" rpy="-0.0 0.0 0.0"/>
-        <parent link="li_top"/>
-        <child link="lidar"/>
-    </joint>
-    <link name="lidar">
-        <visual>
-            <geometry>
-                <cylinder radius="0.06" length="0.04"/>
-            </geometry>
-            <material name="blue"/>
-        </visual>
-        <collision>
-            <geometry>
-                <sphere radius="0.06"/>
-            </geometry>
-        </collision>
-        <xacro:inertial_cylinder mass="0.01" radius="0.06" length="0.04">
-            <origin xyz="0.0 0.0 0.0" rpy="0.0 0.0 0.0"/>
-        </xacro:inertial_cylinder>
-    </link>
 </robot>

Commit message: added pi_rover for transit to jetson nano

File: description/robot.urdf.xacro (robot description, xacro)
@@ -2,6 +2,8 @@
 <robot xmlns:xacro="http://www.ros.org/wiki/xacro"  name="scout">
     <xacro:include filename="robot_core.xacro"/>
+    <!--
     <xacro:include filename="camera.xacro"/>
     <xacro:include filename="lidar.xacro"/>
+    -->
     <xacro:include filename="gazebo_control.xacro"/>
 </robot>

File: description/robot_core.xacro (robot description, xacro)
@@ -34,5 +34,5 @@
         <parent link="base_link"/>
         <child link="chassis"/>
-        <origin xyz="-0.0 0.0 0.0"/>
+        <origin xyz="0.0 0.0 0.0"/>
     </joint>
     <link name="chassis">
@@ -58,5 +58,5 @@
     </gazebo>
     <joint name="chassi_T_joint" type="fixed">
-       <parent link="base_link"/>
+       <parent link="chassis"/>
        <child link="chassis_t"/>
        <origin xyz="-0.12 0.0 0.0"/>
@@ -87,8 +87,8 @@
         <origin xyz="0.0 0.125 0.0" rpy="-${pi/2} 0.0 0.0"/>
         <parent link="base_link"/>
-        <child link="left_wheel"/>
+        <child link="left_wheel_link"/>
         <axis xyz="0.0 0.0 1"/>
     </joint>
-    <link name="left_wheel">
+    <link name="left_wheel_link">
         <visual>
             <geometry>
@@ -106,5 +106,5 @@
         </xacro:inertial_sphere>
     </link>
-    <gazebo reference="left_wheel">
+    <gazebo reference="left_wheel_link">
         <material>Gazebo/Blue</material>
     </gazebo>
@@ -113,8 +113,8 @@
         <origin xyz="0.0 -0.125 0.0" rpy="-${pi/2} 0.0 0.0"/>
         <parent link="base_link"/>
-        <child link="right_wheel"/>
+        <child link="right_wheel_link"/>
         <axis xyz="0.0 0.0 1"/>
     </joint>
-    <link name="right_wheel">
+    <link name="right_wheel_link">
         <visual>
             <geometry>
@@ -132,5 +132,5 @@
         </xacro:inertial_sphere>
     </link>
-    <gazebo reference="right_wheel">
+    <gazebo reference="right_wheel_link">
         <material>Gazebo/Blue</material>
     </gazebo>
@@ -138,5 +138,5 @@
     <joint name="caster_wheel_joint" type="fixed">
         <origin xyz="-0.23 0.0 -0.03" rpy="0.0 0.0 0.0"/>
-        <parent link="base_link"/>
+        <parent link="chassis"/>
         <child link="caster_wheel"/>
     </joint>
@@ -164,5 +164,5 @@
         <!-- Chassis Aufbau-->
     <joint name="body_base_joint" type="fixed">
-        <parent link="base_link"/>
+        <parent link="chassis"/>
         <child link="body"/>
         <origin xyz="-0.08 0.0 0.055"/>

Commit message: next mapping

File: description/robot.urdf.xacro (robot description, xacro)
@@ -1,9 +1,12 @@
 <?xml version="1.0"?>
 <robot xmlns:xacro="http://www.ros.org/wiki/xacro"  name="scout">
-    <xacro:include filename="scout_core.xacro"/>
-    <xacro:include filename="gazebo_control.xacro"/>
-<!--
+    <!-- Argumente -->
     <xacro:arg name="use_ros2_control" default="false"/>
     <xacro:arg name="sim_mode" default="true"/>
+    <!-- Roboter Teile -->
+    <xacro:include filename="robot_core.xacro"/>
+    <xacro:include filename="lidar.xacro"/>
+    <xacro:include filename="camera.xacro"/>
+    <!-- Controller -->
     <xacro:if value="$(arg use_ros2_control)">
         <xacro:include filename="ros2_control.xacro"/>
@@ -12,6 +15,3 @@
         <xacro:include filename="gazebo_control.xacro"/>
     </xacro:unless>
-    <xacro:include filename="lidar.xacro"/>
-    <xacro:include filename="camera.xacro"/>
--->
 </robot>

File: description/robot_core.xacro (robot description, xacro)
@@ -51,5 +51,5 @@
         </visual>
         <collision>
-            <origin xyz="0.093 0.0 0.075"/>
+            <origin xyz="0.017 0.0 0.017"/>
             <geometry>
                 <box size="0.034 0.25 0.034"/>
@@ -89,11 +89,18 @@
     <gazebo reference="left_wheel">
         <material>Gazebo/Blue</material>
+        <mu1 value="100000000000000.0" /><!-- 0.001-->
+        <mu2 value="100000000000000.0" />
+        <kp value="1000000000000.0" />
+        <kd value="10"/>
+        <minDepth>0.001</minDepth>
+        <maxVel>0.1</maxVel>
+        <fdir1>1 0 0</fdir1>
     </gazebo>
     <!-- RIGHT WHEEL  LINK -->
     <joint name="right_wheel_joint" type="continuous">
-        <origin xyz="0 0.128 0.017" rpy="${pi/2} 0 0"/>
+        <origin xyz="0 0.128 0.017" rpy="-${pi/2} 0 0"/>
         <parent link="base_link"/>
         <child link="right_wheel"/>
-        <axis xyz="0.0 0.0 1.0"/>
+        <axis xyz="0.0 0.0 -1.0"/>
         <limit lower="0.0" upper="0.0" effort="0.0" velocity="0.0"/>
     </joint>
@@ -116,8 +123,15 @@
     <gazebo reference="right_wheel">
         <material>Gazebo/Blue</material>
+        <mu1 value="100000000000000.0" /><!-- 0.001-->
+        <mu2 value="100000000000000.0" />
+        <kp value="1000000000000.0" />
+        <kd value="10"/>
+        <minDepth>0.001</minDepth>
+        <maxVel>0.1</maxVel>
+        <fdir1>1 0 0</fdir1>
     </gazebo>
     <!-- Caster Wheel Holder and Caster Wheel -->
     <joint name="caster_wheel_holder_joint" type="fixed">
-        <parent link="chassis"/>
+        <parent link="base_link"/>
         <child link="caster_wheel_holder"/>
         <origin xyz="0.25 0.0 0.0"/>
@@ -169,6 +183,11 @@
     <gazebo reference="caster_wheel_link">
         <material>Gazebo/Blue</material>
-        <mu1 value="0.001"/>
-        <mu2 value="0.001"/>
+        <mu1 value="100000000000000.0" /><!-- 0.001-->
+        <mu2 value="100000000000000.0" />
+        <kp value="1000000000000.0" />
+        <kd value="10"/>
+        <minDepth>0.001</minDepth>
+        <maxVel>0.1</maxVel>
+        <fdir1>1 0 0</fdir1>
     </gazebo>
     <!-- BODY PARTS-->

File: description/ros2_control.xacro (robot description, xacro)
@@ -32,4 +32,23 @@
     </xacro:unless>
     <xacro:if value="$(arg sim_mode)">
+        <gazebo>
+        <plugin name="diff_drive" filename="libgazebo_ros_diff_drive.so">
+            <!-- Reifen Infos -->
+            <left_joint>left_wheel_joint</left_joint>
+            <right_joint>right_wheel_joint</right_joint>
+            <wheel_separation>0.3</wheel_separation>
+            <wheel_diameter>0.12</wheel_diameter>
+            <!-- LIMITS       -->
+            <max_wheel_torque>200</max_wheel_torque>
+            <max_wheel_acceleration>10.0</max_wheel_acceleration>
+            <!-- Output       -->
+            <odometry_frame>odom</odometry_frame>
+            <robot_base_frame>base_link</robot_base_frame>
+            <publish_odom>true</publish_odom>
+            <publish_odom_tf>true</publish_odom_tf>
+            <publish_wheel_tf>true</publish_wheel_tf>
+        </plugin>
+        </gazebo>
+    <!--
         <ros2_control name="GazeboSystem" type="system">
             <hardware>
@@ -52,5 +71,5 @@
                 <state_interface name="position"/>
             </joint>
-        </ros2_control>
+        </ros2_control> -->
     </xacro:if>
     <gazebo>
