Commit message: fehler suche odom--base_link-

File: description/camera.xacro (robot description, xacro)
@@ -24,4 +24,7 @@
             <origin xyz="0.0 0.0 0.0" rpy="0.0 0.0 0.0"/>
         </xacro:inertial_box>
-     </link>
+    </link>
+    <gazebo reference="cam">
+        <material>Gazebo/White</material>
+    </gazebo>
 </robot>

File: description/lidar.xacro (robot description, xacro)
@@ -1,6 +1,6 @@
 <?xml version="1.0"?>
 <robot xmlns:xacro="http://www.ros.org/wiki/xacro">
-     <!-- LIDAR-->
-     <joint name="li_top_joint" type="fixed">
+    <!-- LIDAR-->
+    <joint name="li_top_joint" type="fixed">
         <parent link="body_top"/>
         <child link="li_top"/>
@@ -24,9 +24,12 @@
             <origin xyz="0.0 0.0 0.0" rpy="0.0 0.0 0.0"/>
         </xacro:inertial_box>
-     </link>
-     <joint name="lidar_joint" type="fixed">
-        <origin xyz="0.0 0.0 0.03" rpy="-0.0 0.0 0.0"/>
-        <parent link="li_top"/>
-        <child link="lidar"/>
+    </link>
+    <gazebo reference="li_top">
+        <material>Gazebo/Black</material>
+    </gazebo>
+    <joint name="lidar_joint" type="fixed">
+       <origin xyz="0.0 0.0 0.03" rpy="-0.0 0.0 0.0"/>
+       <parent link="li_top"/>
+       <child link="lidar"/>
     </joint>
     <link name="lidar">
@@ -39,5 +42,5 @@
         <collision>
             <geometry>
-                <sphere radius="0.06"/>
+                <cylinder radius="0.06" length="0.04"/>
             </geometry>
         </collision>
@@ -46,3 +49,6 @@
         </xacro:inertial_cylinder>
     </link>
+    <gazebo reference="lidar">
+        <material>Gazebo/Red</material>
+    </gazebo>
 </robot>

File: description/robot.urdf.xacro (robot description, xacro)
@@ -4,3 +4,4 @@
     <xacro:include filename="camera.xacro"/>
     <xacro:include filename="lidar.xacro"/>
+    <xacro:include filename="gazebo_control.xacro"/>
 </robot>

File: description/robot_core.xacro (robot description, xacro)
@@ -32,6 +32,6 @@
     <!-- Chassis Link AKA Rad Strebe-->
     <joint name="chassis_joint" type="fixed">
-        <parent link="chassis"/>
-        <child link="base_link"/>
+        <parent link="base_link"/>
+        <child link="chassis"/>
         <origin xyz="-0.0 0.0 0.0"/>
     </joint>
@@ -50,12 +50,15 @@
             </geometry>
         </collision>
-        <xacro:inertial_box mass="0.5" x="0.034" y="0.025" z="0.034">
-            <origin xyz="0.0 0.0 0.003" rpy="0.0 0.0 0.0"/>
-        </xacro:inertial_box>
-     </link>
-     <joint name="chassi_T_joint" type="fixed">
-        <parent link="base_link"/>
-        <child link="chassis_t"/>
-        <origin xyz="-0.12 0.0 0.0"/>
+        <xacro:inertial_box mass="1.5" x="0.034" y="0.025" z="0.034">
+            <origin xyz="0.0 0.0 0.003" rpy="0.0 0.0 0.0"/>
+        </xacro:inertial_box>
+    </link>
+    <gazebo reference="chassis">
+        <material>Gazebo/Black</material>
+    </gazebo>
+    <joint name="chassi_T_joint" type="fixed">
+       <parent link="base_link"/>
+       <child link="chassis_t"/>
+       <origin xyz="-0.12 0.0 0.0"/>
     </joint>
     <link name="chassis_t">
@@ -73,8 +76,11 @@
             </geometry>
         </collision>
-        <xacro:inertial_box mass="0.5" x="0.034" y="0.025" z="0.034">
-            <origin xyz="0.0 0.0 0.003" rpy="0.0 0.0 0.0"/>
-        </xacro:inertial_box>
-     </link>
+        <xacro:inertial_box mass="1.5" x="0.034" y="0.025" z="0.034">
+            <origin xyz="0.0 0.0 0.003" rpy="0.0 0.0 0.0"/>
+        </xacro:inertial_box>
+    </link>
+    <gazebo reference="chassis_t">
+        <material>Gazebo/Black</material>
+    </gazebo>
     <!-- Linker Reifen-->
     <joint name="left_wheel_joint" type="continuous">
@@ -100,4 +106,7 @@
         </xacro:inertial_sphere>
     </link>
+    <gazebo reference="left_wheel">
+        <material>Gazebo/Blue</material>
+    </gazebo>
     <!-- Rechter Reifen-->
     <joint name="right_wheel_joint" type="continuous">
@@ -123,4 +132,7 @@
         </xacro:inertial_sphere>
     </link>
+    <gazebo reference="right_wheel">
+        <material>Gazebo/Blue</material>
+    </gazebo>
     <!-- Caster Wheel Joint-->
     <joint name="caster_wheel_joint" type="fixed">
@@ -134,5 +146,5 @@
                 <sphere radius="0.03"/>
             </geometry>
-            <material name="LightGrey"/>
+            <material name="blue"/>
         </visual>
         <collision>
@@ -145,4 +157,9 @@
         </xacro:inertial_sphere>
     </link>
+    <gazebo reference="caster_wheel">
+        <material>Gazebo/Blue</material>
+        <mu1 value="0.001"/>
+        <mu2 value="0.001"/>
+    </gazebo>
         <!-- Chassis Aufbau-->
     <joint name="body_base_joint" type="fixed">
@@ -168,6 +185,9 @@
             <origin xyz="0.0 0.0 0.003" rpy="0.0 0.0 0.0"/>
         </xacro:inertial_box>
-     </link>
-     <joint name="body_joint" type="fixed">
+    </link>
+    <gazebo reference="body">
+        <material>Gazebo/Orange</material>
+    </gazebo>
+    <joint name="body_joint" type="fixed">
         <parent link="body"/>
         <child link="body_top"/>
@@ -191,4 +211,7 @@
             <origin xyz="0.0 0.0 0.0" rpy="0.0 0.0 0.0"/>
         </xacro:inertial_box>
-     </link>
+    </link>
+    <gazebo reference="body_top">
+        <material>Gazebo/Orange</material>
+    </gazebo>
 </robot>

Commit message: working on lidar

File: description/camera.xacro (robot description, xacro)
@@ -29,5 +29,5 @@
     </gazebo>
     <gazebo reference="cam">
-        <material>Gazebo/Orange</material>
+        <material>Gazebo/White</material>
         <sensor name="camera" type="camera">
             <pose> 0 0 0 0 0 0 </pose>

File: description/gazebo_control.xacro (robot description, xacro)
@@ -6,5 +6,5 @@
             <left_joint>left_wheel_joint</left_joint>
             <right_joint>right_wheel_joint</right_joint>
-            <wheel_separation>0.35</wheel_separation>
+            <wheel_separation>0.36</wheel_separation>
             <wheel_diameter>0.12</wheel_diameter>
             <!-- LIMITS       -->

File: description/lidar.xacro (robot description, xacro)
@@ -29,5 +29,5 @@
     </gazebo>
     <joint name="lidar_joint" type="fixed">
-       <origin xyz="0.0 0.0 0.03" rpy="-0.0 0.0 0.0"/>
+       <origin xyz="0.0 0.0 0.03" rpy="0.0 0.0 1.57"/>
        <parent link="li_top"/>
        <child link="lidar"/>
@@ -67,10 +67,11 @@
                 <range>
                     <min>0.3</min>
-                    <max>8</max>
+                    <max>12</max>
+                    <resolution>0.01</resolution>
                 </range>
             </ray>
             <plugin name="laser_controller" filename="libgazebo_ros_ray_sensor.so">
                 <ros>
-                    <argument>~/out:=scan</argument>
+                    <argument>~/out:=scan</argument> <!-- - -ros-args - -remap ~ -->
                 </ros>
                 <output_type>sensor_msgs/LaserScan</output_type>

File: description/robot.urdf.xacro (robot description, xacro)
@@ -11,4 +11,6 @@
     </xacro:unless>
     <xacro:include filename="lidar.xacro"/>
+<!--
     <xacro:include filename="camera.xacro"/>
+-->
 </robot>

File: description/robot_core.xacro (robot description, xacro)
@@ -71,10 +71,10 @@
         <collision>
             <geometry>
-                <cylinder radius="0.06" length="0.04"/>
-            </geometry>
-        </collision>
-        <xacro:inertial_cylinder mass="0.1" length="0.04" radius="0.06">
-            <origin xyz="0.0 0.0 0.0" rpy="0.0 0.0 0.0"/>
-        </xacro:inertial_cylinder>
+                <sphere radius="0.06"/>
+            </geometry>
+        </collision>
+        <xacro:inertial_sphere mass="0.3" radius="0.06">
+            <origin xyz="0.0 0.0 0.0" rpy="0.0 0.0 0.0"/>
+        </xacro:inertial_sphere>
     </link>
     <gazebo reference="left_wheel">
@@ -98,10 +98,10 @@
         <collision>
             <geometry>
-                <cylinder radius="0.06" length="0.04"/>
-            </geometry>
-        </collision>
-        <xacro:inertial_cylinder mass="0.1" length="0.04" radius="0.06">
-            <origin xyz="0.0 0.0 0.0" rpy="0.0 0.0 0.0"/>
-        </xacro:inertial_cylinder>
+                <sphere radius="0.06"/>
+            </geometry>
+        </collision>
+        <xacro:inertial_sphere mass="0.3" radius="0.06">
+            <origin xyz="0.0 0.0 0.0" rpy="0.0 0.0 0.0"/>
+        </xacro:inertial_sphere>
     </link>
     <gazebo reference="right_wheel">

Commit message: cam in gazebo in work

File: description/camera.xacro (robot description, xacro)
@@ -2,10 +2,10 @@
 <robot xmlns:xacro="http://www.ros.org/wiki/xacro">
     <!-- Cam-->
-    <joint name="cam_joint" type="fixed">
+    <joint name="camera_joint" type="fixed">
         <parent link="chassis"/>
-        <child link="cam"/>
+        <child link="camera_link"/>
         <origin xyz="-0.04 0 0.138 "/>
     </joint>
-    <link name="cam">
+    <link name="camera_link">
         <visual>
             <origin xyz="0.0 0.0 0.0" rpy="0.0 0.0 0.0"/>
@@ -25,8 +25,14 @@
         </xacro:inertial_box>
     </link>
-    <gazebo reference="cam">
+    <gazebo reference="camera_link">
         <material>Gazebo/White</material>
     </gazebo>
-    <gazebo reference="cam">
+    <joint name="cam_joint" type="fixed">
+        <parent link="camera_link"/>
+        <child link="camera_link_optocal"/>
+        <origin xyz="0 0 0" rpy="${-pi/2} 0.0 ${-pi/2}"/>
+    </joint>
+    <link name="camera_link_optical"/>
+    <gazebo reference="camera_link">
         <material>Gazebo/White</material>
         <sensor name="camera" type="camera">

File: description/robot.urdf.xacro (robot description, xacro)
@@ -11,6 +11,4 @@
     </xacro:unless>
     <xacro:include filename="lidar.xacro"/>
-<!--
     <xacro:include filename="camera.xacro"/>
--->
 </robot>

Commit message: cam in gazebo works fine

File: description/camera.xacro (robot description, xacro)
@@ -5,5 +5,5 @@
         <parent link="chassis"/>
         <child link="camera_link"/>
-        <origin xyz="-0.04 0 0.138 "/>
+        <origin xyz="-0.04 0 0.138 " rpy="0.0 0.0 3.14"/>
     </joint>
     <link name="camera_link">
@@ -30,6 +30,6 @@
     <joint name="cam_joint" type="fixed">
         <parent link="camera_link"/>
-        <child link="camera_link_optocal"/>
-        <origin xyz="0 0 0" rpy="${-pi/2} 0.0 ${-pi/2}"/>
+        <child link="camera_link_optical"/>
+        <origin xyz="0.0 0.0 0.0" rpy="0.0 0.0 0.0"/>
     </joint>
     <link name="camera_link_optical"/>
@@ -49,5 +49,5 @@
                 <clip>
                     <near>0.05</near>
-                    <far>7.0</far>
+                    <far>8.0</far>
                 </clip>
             </camera>

File: description/lidar.xacro (robot description, xacro)
@@ -57,5 +57,5 @@
         <sensor name="laser" type="ray">
             <pose> 0 0 0 0 0 0 </pose>
-            <visualize>true</visualize>
+            <visualize>false</visualize>
             <update_rate>10</update_rate>
             <ray>

Commit message: change some thinges in the urdf files

File: description/camera.xacro (robot description, xacro)
@@ -3,7 +3,7 @@
     <!-- Cam-->
     <joint name="camera_joint" type="fixed">
-        <parent link="chassis"/>
+        <parent link="base_link"/>
         <child link="camera_link"/>
-        <origin xyz="-0.04 0 0.138 " rpy="0.0 0.0 3.14"/>
+        <origin xyz="0.1 0 0.14 " rpy="0.0 0.0 0.0"/>
     </joint>
     <link name="camera_link">

File: description/lidar.xacro (robot description, xacro)
@@ -5,5 +5,5 @@
         <parent link="body_top"/>
         <child link="li_top"/>
-        <origin xyz="-0.12 0 0.047 "/>
+        <origin xyz="0.12 0 0.047 "/>
     </joint>
     <link name="li_top">
@@ -29,5 +29,5 @@
     </gazebo>
     <joint name="lidar_joint" type="fixed">
-       <origin xyz="0.0 0.0 0.03" rpy="0.0 0.0 1.57"/>
+       <origin xyz="0.0 0.0 0.03" rpy="0.0 0.0 -1.57"/>
        <parent link="li_top"/>
        <child link="laser_frame"/>

File: description/robot.urdf.xacro (robot description, xacro)
@@ -1,11 +1,11 @@
 <?xml version="1.0"?>
 <robot xmlns:xacro="http://www.ros.org/wiki/xacro"  name="scout">
-    <!-- Argumente -->
+    <!-- Argumente-->
     <xacro:arg name="use_ros2_control" default="false"/>
     <xacro:arg name="sim_mode" default="true"/>
     <!-- Roboter Teile -->
-    <xacro:include filename="robot_core.xacro"/>
+    <xacro:include filename="scout_core.xacro"/>
+    <xacro:include filename="camera.xacro"/>
     <xacro:include filename="lidar.xacro"/>
-    <xacro:include filename="camera.xacro"/>
     <!-- Controller -->
     <xacro:if value="$(arg use_ros2_control)">

File: description/scout_core.xacro (robot description, xacro)
@@ -163,3 +163,57 @@
         <mu2 value="0.001"/>
     </gazebo>
+    <!-- BODY PARTS-->
+    <joint name="body_joint" type="fixed">
+        <parent link="base_link"/>
+        <child link="body"/>
+        <origin xyz="-0.065 0.0 0.069"/>
+    </joint>
+    <link name="body">
+        <visual>
+            <origin xyz="0.0 0.0 0.0"/>
+            <geometry>
+                <box size="0.4 0.11 0.07"/>
+            </geometry>
+            <material name="orange"/>
+        </visual>
+        <collision>
+            <origin xyz="0.0 0.0 0.0"/>
+            <geometry>
+                <box size="0.4 0.11 0.07"/>
+            </geometry>
+        </collision>
+        <xacro:inertial_box mass="0.5" x="0.4" y="0.11" z="0.07">
+            <origin xyz="0.0 0.0 0.0" rpy="0.0 0.0 0.0"/>
+        </xacro:inertial_box>
+    </link>
+    <gazebo reference="body">
+        <material>Gazebo/Orange</material>
+    </gazebo>
+    <!-- BodyTop-->
+    <joint name="body_top_joint" type="fixed">
+        <parent link="body"/>
+        <child link="body_top"/>
+        <origin xyz="-0.05 0.0 0.07"/>
+    </joint>
+    <link name="body_top">
+        <visual>
+            <origin xyz="0.0 0.0 0.0"/>
+            <geometry>
+                <box size="0.3 0.11 0.07"/>
+            </geometry>
+            <material name="orange"/>
+        </visual>
+        <collision>
+            <origin xyz="0.0 0.0 0.0"/>
+            <geometry>
+                <box size="0.3 0.11 0.07"/>
+            </geometry>
+        </collision>
+        <xacro:inertial_box mass="0.5" x="0.3" y="0.11" z="0.07">
+            <origin xyz="0.0 0.0 0.0" rpy="0.0 0.0 0.0"/>
+        </xacro:inertial_box>
+    </link>
+    <gazebo reference="body_top">
+        <material>Gazebo/Orange</material>
+    </gazebo>
 </robot>
